Commit message: modified URDF files

File: Hardware/URDF/robots/Heol_humanoid.URDF (robot description, URDF)
Before this commit: robot Fendi_humanoid, 24 links, 23 joints
Links:
- link chest: mass 0.0758588949423129 -> 0.08200767006894; geometry collision mesh filename=package://Heol_humanoid/meshes/chest.STL; visual mesh filename=package://Heol_humanoid/meshes/chest.STL
- link head: mass 0.0229562091454423 -> 0.0234153108401363; geometry collision mesh filename=package://Heol_humanoid/meshes/head.STL; visual mesh filename=package://Heol_humanoid/meshes/head.STL
- link l_ankle: geometry collision mesh filename=package://Heol_humanoid/meshes/l_ankle.STL; visual mesh filename=package://Heol_humanoid/meshes/l_ankle.STL
- link l_foot: geometry collision mesh filename=package://Heol_humanoid/meshes/l_foot.STL; visual mesh filename=package://Heol_humanoid/meshes/l_foot.STL
- link l_forearm: geometry collision mesh filename=package://Heol_humanoid/meshes/l_forearm.STL; visual mesh filename=package://Heol_humanoid/meshes/l_forearm.STL
- link l_hip: geometry collision mesh filename=package://Heol_humanoid/meshes/l_hip.STL; visual mesh filename=package://Heol_humanoid/meshes/l_hip.STL
- link l_hip_motor: geometry collision mesh filename=package://Heol_humanoid/meshes/l_hip_motor.STL; visual mesh filename=package://Heol_humanoid/meshes/l_hip_motor.STL
- link l_knee: geometry collision mesh filename=package://Heol_humanoid/meshes/l_knee.STL; visual mesh filename=package://Heol_humanoid/meshes/l_knee.STL
- link l_shoulder: geometry collision mesh filename=package://Heol_humanoid/meshes/l_shoulder.STL; visual mesh filename=package://Heol_humanoid/meshes/l_shoulder.STL
- link l_shoulder_motor: geometry collision mesh filename=package://Heol_humanoid/meshes/l_shoulder_motor.STL; visual mesh filename=package://Heol_humanoid/meshes/l_shoulder_motor.STL
- link l_thigh: mass 0.0205479194607194 -> 0.0205479105964943; geometry collision mesh filename=package://Heol_humanoid/meshes/l_thigh.STL; visual mesh filename=package://Heol_humanoid/meshes/l_thigh.STL
- link l_upper_arm: mass 0.00334368326578746 -> 0.00334368326578747; geometry collision mesh filename=package://Heol_humanoid/meshes/l_upper_arm.STL; visual mesh filename=package://Heol_humanoid/meshes/l_upper_arm.STL
- link pelvis: geometry collision mesh filename=package://Heol_humanoid/meshes/pelvis.STL; visual mesh filename=package://Heol_humanoid/meshes/pelvis.STL
- link r_ankle: geometry collision mesh filename=package://Heol_humanoid/meshes/r_ankle.STL; visual mesh filename=package://Heol_humanoid/meshes/r_ankle.STL
- link r_foot: geometry collision mesh filename=package://Heol_humanoid/meshes/r_foot.STL; visual mesh filename=package://Heol_humanoid/meshes/r_foot.STL
- link r_forearm: geometry collision mesh filename=package://Heol_humanoid/meshes/r_forearm.STL; visual mesh filename=package://Heol_humanoid/meshes/r_forearm.STL
- link r_hip: geometry collision mesh filename=package://Heol_humanoid/meshes/r_hip.STL; visual mesh filename=package://Heol_humanoid/meshes/r_hip.STL
- link r_hip_motor: geometry collision mesh filename=package://Heol_humanoid/meshes/r_hip_motor.STL; visual mesh filename=package://Heol_humanoid/meshes/r_hip_motor.STL
- link r_knee: geometry collision mesh filename=package://Heol_humanoid/meshes/r_knee.STL; visual mesh filename=package://Heol_humanoid/meshes/r_knee.STL
- link r_shoulder: mass 0.00334368326561427 -> 0.00334368326561429; geometry collision mesh filename=package://Heol_humanoid/meshes/r_shoulder.STL; visual mesh filename=package://Heol_humanoid/meshes/r_shoulder.STL
- link r_shoulder_motor: mass 0.0337180938564699 -> 0.0337180938758863; geometry collision mesh filename=package://Heol_humanoid/meshes/r_shoulder_motor.STL; visual mesh filename=package://Heol_humanoid/meshes/r_shoulder_motor.STL
- link r_thigh: geometry collision mesh filename=package://Heol_humanoid/meshes/r_thigh.STL; visual mesh filename=package://Heol_humanoid/meshes/r_thigh.STL
- link r_upper_arm: mass 0.00334368326578747 -> 0.00334368326578746; geometry collision mesh filename=package://Heol_humanoid/meshes/r_upper_arm.STL; visual mesh filename=package://Heol_humanoid/meshes/r_upper_arm.STL
- link spine: mass 0.0236192598262426 -> 0.0236192598262425; geometry collision mesh filename=package://Heol_humanoid/meshes/spine.STL; visual mesh filename=package://Heol_humanoid/meshes/spine.STL
Joints:
- joint chest_x: limit (none) -> lower=-2.6 upper=2.6 effort=0 velocity=0; origin xyz=0 0.0150000000000001 0 rpy=-1.5707963267949 0 0 -> xyz=0 0.015 0 rpy=-1.5708 0 0
- joint head_z: limit (none) -> lower=-2.6 upper=2.6 effort=0 velocity=0; origin xyz=0.00020516550046587 -0.00211629613324466 0.0760159797629514 rpy=1.59665875812253 6.47649529920312E-05 -6.311126761483E-05 -> xyz=0.00020517 -0.0021163 0.076016 rpy=1.5967 6.4765E-05 -6.3111E-05
- joint l_ankle_x: limit (none) -> lower=-2.6 upper=2.6 effort=0 velocity=0; origin xyz=0 0.0450000000000011 0 rpy=3.46944695195361E-16 0 3.14159265358979 -> xyz=0 0.045 0 rpy=3.4694E-16 0 3.1416
- joint l_foot_y: limit (none) -> lower=-2.6 upper=2.6 effort=0 velocity=0; origin xyz=0 0 -0.000199999999993367 rpy=2.94902990916057E-15 0 3.14159265358979 -> xyz=0 0 -0.0002 rpy=2.949E-15 0 3.1416
- joint l_forearm_y: limit (none) -> lower=-2.6 upper=2.6 effort=0 velocity=0; origin xyz=0.0179999999999999 0 0 rpy=3.14159265358977 1.11022302462516E-14 -1.5707963267949 -> xyz=0.018 0 0 rpy=3.1416 1.1102E-14 -1.5708
- joint l_hip_motor_z: limit (none) -> lower=-2.6 upper=2.6 effort=0 velocity=0; origin xyz=-0.0319999999999984 0.03 0 rpy=0 0 0 -> xyz=-0.032 0.03 0 rpy=0 0 0
- joint l_hip_y: limit (none) -> lower=-2.6 upper=2.6 effort=0 velocity=0; origin xyz=0.0416518518525676 -0.0188002160308141 0.0267433423130832 rpy=1.5707963267949 0 0 -> xyz=0.041652 -0.0188 0.026743 rpy=1.5708 0 0
- joint l_knee_x: limit (none) -> lower=-2.6 upper=2.6 effort=0 velocity=0; origin xyz=0 -0.0449999999999764 0 rpy=-3.14159265358979 0 0 -> xyz=0 -0.045 0 rpy=-3.1416 0 0; type continuous -> revolute
- joint l_shoulder_motor_y: limit (none) -> lower=-2.6 upper=2.6 effort=0 velocity=0; origin xyz=0.0179999999999996 0 0 rpy=0 -7.88860905221039E-31 0 -> xyz=0.018 0 0 rpy=0 -7.8886E-31 0
- joint l_shoulder_x: limit (none) -> lower=-2.6 upper=2.6 effort=0 velocity=0; origin xyz=-0.0436000000000003 -0.000150337590467807 0.0510000000000027 rpy=1.57079632679489 -1.30000271246138E-29 3.14159265358979 -> xyz=-0.0436 -0.00015034 0.051 rpy=1.5708 -1.3E-29 3.1416
- joint l_thigh_x: limit (none) -> lower=-2.6 upper=2.6 effort=0 velocity=0; origin xyz=0 0 -0.00400000000000341 rpy=1.5707963267949 0 1.5707963267949 -> xyz=0 0 -0.004 rpy=1.5708 0 1.5708
- joint l_upper_arm_z: limit (none) -> lower=-2.6 upper=2.6 effort=0 velocity=0; origin xyz=0 -0.0539999999999975 0 rpy=3.14159265358978 2.08166817117217E-15 -1.5707963267949 -> xyz=0 -0.054 0 rpy=3.1416 2.0817E-15 -1.5708
- joint r_ankle_x: limit (none) -> lower=-2.6 upper=2.6 effort=0 velocity=0; origin xyz=0 -0.0450000000000004 0 rpy=-3.14159265358979 1.38777878078145E-15 3.14159265358979 -> xyz=0 -0.045 0 rpy=-3.1416 1.3878E-15 3.1416
- joint r_foot_y: limit (none) -> lower=-2.6 upper=2.6 effort=0 velocity=0; origin xyz=0 0 -0.000199999999999714 rpy=1.38777878078145E-15 8.32667268468867E-15 3.14159265358979 -> xyz=0 0 -0.0002 rpy=1.3878E-15 8.3267E-15 3.1416
- joint r_forearm_y: limit (none) -> lower=-2.6 upper=2.6 effort=0 velocity=0; origin xyz=0.0180000000000033 0 0 rpy=-3.14159265358979 2.08166817117217E-14 -1.5707963267949 -> xyz=0.018 0 0 rpy=-3.1416 2.0817E-14 -1.5708
- joint r_hip_motor_z: limit (none) -> lower=-2.6 upper=2.6 effort=0 velocity=0; origin xyz=0.0319999970253307 0.053 0 rpy=0 0 0 -> xyz=0.032 0.053 0 rpy=0 0 0
- joint r_hipy: limit (none) -> lower=-2.6 upper=2.6 effort=0 velocity=0; origin xyz=0.0416518518525676 -0.0188002160308141 0.00374334231308317 rpy=1.5707963267949 0 0 -> xyz=0.041652 -0.0188 0.0037433 rpy=1.5708 0 0
- joint r_knee_x: limit (none) -> lower=-2.6 upper=2.6 effort=0 velocity=0; origin xyz=0 -0.0450000000000016 0 rpy=1.38777878078145E-15 1.38777878078145E-15 1.34815096107107E-29 -> xyz=0 -0.045 0 rpy=1.3878E-15 1.3878E-15 1.3482E-29
- joint r_shoulder_motor_y: limit (none) -> lower=-2.6 upper=2.6 effort=0 velocity=0; origin xyz=0.0180885762087062 0 0 rpy=-9.86076131526265E-32 4.33680868994203E-19 3.14159265358979 -> xyz=0.018089 0 0 rpy=-9.8608E-32 4.3368E-19 3.1416
- joint r_shoulder_x: limit (none) -> lower=-2.6 upper=2.6 effort=0 velocity=0; origin xyz=0.0439112930179202 0.000107167499561404 0.0510002215817856 rpy=-1.5707963267949 -1.69346344342082E-18 0.00244054044922089 -> xyz=0.043911 0.00010717 0.051 rpy=-1.5708 -1.6935E-18 0.0024405
- joint r_thigh_x: limit (none) -> lower=-2.6 upper=2.6 effort=0 velocity=0; origin xyz=0 0 -0.00399999999999812 rpy=1.5707963267949 0 1.57079632679491 -> xyz=0 0 -0.004 rpy=1.5708 0 1.5708
- joint r_upper_arm_z: limit (none) -> lower=-2.6 upper=2.6 effort=0 velocity=0; origin xyz=0 -0.0539999999999969 0 rpy=-3.13915211314058 6.9388732390668E-16 -1.5707963267949 -> xyz=0 -0.054 0 rpy=-3.1392 6.9389E-16 -1.5708
- joint spine_z: limit (none) -> lower=-2.6 upper=2.6 effort=0 velocity=0; origin xyz=0.0416518518525676 -0.0728002160308141 0.0587433423130832 rpy=3.14159265358979 0 0 -> xyz=0.041652 -0.0728 0.058743 rpy=3.1416 0 0

Commit message: add vrep scene

File: Hardware/URDF/robots/Heol_humanoid.URDF (robot description, URDF)
Before this commit: robot Heol_humanoid, 24 links, 23 joints
Links:
- link chest: geometry collision mesh filename=package://meshes/chest_respondable.STL; visual mesh filename=package://meshes/chest_visual.STL
- link head: geometry collision mesh filename=package://meshes/head_respondable.STL; visual mesh filename=package://meshes/head_visual.STL
- link l_ankle: geometry collision mesh filename=package://meshes/l_ankle_respondable.STL; visual mesh filename=package://meshes/l_ankle_visual.STL
- link l_foot: geometry collision mesh filename=package://meshes/l_foot_respondable.STL; visual mesh filename=package://meshes/l_foot_visual.STL
- link l_forearm: geometry collision mesh filename=package://meshes/l_forearm_respondable.STL; visual mesh filename=package://meshes/l_forearm_visual.STL
- link l_hip: geometry collision mesh filename=package://meshes/l_hip_respondable.STL; visual mesh filename=package://meshes/l_hip_visual.STL
- link l_hip_motor: geometry collision mesh filename=package://meshes/l_hip_motor_respondable.STL; visual mesh filename=package://meshes/l_hip_motor_visual.STL
- link l_knee: geometry collision mesh filename=package://meshes/l_knee_respondable.STL; visual mesh filename=package://meshes/l_knee_visual.STL
- link l_shoulder: geometry collision mesh filename=package://meshes/l_shoulder_respondable.STL; visual mesh filename=package://meshes/l_shoulder_visual.STL
- link l_shoulder_motor: geometry collision mesh filename=package://meshes/l_shoulder_motor_respondable.STL; visual mesh filename=package://meshes/l_shoulder_motor_visual.STL
- link l_thigh: geometry collision mesh filename=package://meshes/l_thigh_respondable.STL; visual mesh filename=package://meshes/l_thigh_visual.STL
- link l_upper_arm: geometry collision mesh filename=package://meshes/l_upper_arm_respondable.STL; visual mesh filename=package://meshes/l_upper_arm_visual.STL
- link pelvis: geometry collision mesh filename=package://meshes/pelvis_respondable.STL; visual mesh filename=package://meshes/pelvis_visual.STL
- link r_ankle: geometry collision mesh filename=package://meshes/r_ankle_respondable.STL; visual mesh filename=package://meshes/r_ankle_visual.STL
- link r_foot: geometry collision mesh filename=package://meshes/r_foot_respondable.STL; visual mesh filename=package://meshes/r_foot_visual.STL
- link r_forearm: geometry collision mesh filename=package://meshes/r_forearm_respondable.STL; visual mesh filename=package://meshes/r_forearm_visual.STL
- link r_hip: geometry collision mesh filename=package://meshes/r_hip_respondable.STL; visual mesh filename=package://meshes/r_hip_visual.STL
- link r_hip_motor: geometry collision mesh filename=package://meshes/r_hip_motor_respondable.STL; visual mesh filename=package://meshes/r_hip_motor_visual.STL
- link r_knee: geometry collision mesh filename=package://meshes/r_knee_respondable.STL; visual mesh filename=package://meshes/r_knee_visual.STL
- link r_shoulder: geometry collision mesh filename=package://meshes/r_shoulder_respondable.STL; visual mesh filename=package://meshes/r_shoulder_visual.STL
- link r_shoulder_motor: geometry collision mesh filename=package://meshes/r_shoulder_motor_respondable.STL; visual mesh filename=package://meshes/r_shoulder_motor_visual.STL
- link r_thigh: geometry collision mesh filename=package://meshes/r_thigh_respondable.STL; visual mesh filename=package://meshes/r_thigh_visual.STL
- link r_upper_arm: geometry collision mesh filename=package://meshes/r_upper_arm_respondable.STL; visual mesh filename=package://meshes/r_upper_arm_visual.STL
- link spine: geometry collision mesh filename=package://meshes/spine_respondable.STL; visual mesh filename=package://meshes/spine_visual.STL
Joints:
- joint chest_x: limit lower=-2.6 upper=2.6 effort=0 velocity=0 -> lower=-2.6 upper=2.6 effort=3.1 velocity=7.0
- joint head_z: limit lower=-2.6 upper=2.6 effort=0 velocity=0 -> lower=-2.6 upper=2.6 effort=3.1 velocity=7.0
- joint l_ankle_x: limit lower=-2.6 upper=2.6 effort=0 velocity=0 -> lower=-2.6 upper=2.6 effort=3.1 velocity=7.0
- joint l_foot_y: limit lower=-2.6 upper=2.6 effort=0 velocity=0 -> lower=-2.6 upper=2.6 effort=3.1 velocity=7.0
- joint l_forearm_y: limit lower=-2.6 upper=2.6 effort=0 velocity=0 -> lower=-2.6 upper=2.6 effort=3.1 velocity=7.0
- joint l_hip_motor_z: limit lower=-2.6 upper=2.6 effort=0 velocity=0 -> lower=-2.6 upper=2.6 effort=3.1 velocity=7.0
- joint l_hip_y: limit lower=-2.6 upper=2.6 effort=0 velocity=0 -> lower=-2.6 upper=2.6 effort=3.1 velocity=7.0
- joint l_knee_x: limit lower=-2.6 upper=2.6 effort=0 velocity=0 -> lower=-2.6 upper=2.6 effort=3.1 velocity=7.0
- joint l_shoulder_motor_y: limit lower=-2.6 upper=2.6 effort=0 velocity=0 -> lower=-2.6 upper=2.6 effort=3.1 velocity=7.0
- joint l_shoulder_x: limit lower=-2.6 upper=2.6 effort=0 velocity=0 -> lower=-2.6 upper=2.6 effort=3.1 velocity=7.0
- joint l_thigh_x: limit lower=-2.6 upper=2.6 effort=0 velocity=0 -> lower=-2.6 upper=2.6 effort=3.1 velocity=7.0
- joint l_upper_arm_z: limit lower=-2.6 upper=2.6 effort=0 velocity=0 -> lower=-2.6 upper=2.6 effort=3.1 velocity=7.0
- joint r_ankle_x: limit lower=-2.6 upper=2.6 effort=0 velocity=0 -> lower=-2.6 upper=2.6 effort=3.1 velocity=7.0
- joint r_foot_y: limit lower=-2.6 upper=2.6 effort=0 velocity=0 -> lower=-2.6 upper=2.6 effort=3.1 velocity=7.0
- joint r_forearm_y: limit lower=-2.6 upper=2.6 effort=0 velocity=0 -> lower=-2.6 upper=2.6 effort=3.1 velocity=7.0
- joint r_hip_motor_z: limit lower=-2.6 upper=2.6 effort=0 velocity=0 -> lower=-2.6 upper=2.6 effort=3.1 velocity=7.0
- joint r_hipy: limit lower=-2.6 upper=2.6 effort=0 velocity=0 -> lower=-2.6 upper=2.6 effort=3.1 velocity=7.0
- joint r_knee_x: limit lower=-2.6 upper=2.6 effort=0 velocity=0 -> lower=-2.6 upper=2.6 effort=3.1 velocity=7.0
- joint r_shoulder_motor_y: limit lower=-2.6 upper=2.6 effort=0 velocity=0 -> lower=-2.6 upper=2.6 effort=3.1 velocity=7.0
- joint r_shoulder_x: limit lower=-2.6 upper=2.6 effort=0 velocity=0 -> lower=-2.6 upper=2.6 effort=3.1 velocity=7.0
- joint r_thigh_x: limit lower=-2.6 upper=2.6 effort=0 velocity=0 -> lower=-2.6 upper=2.6 effort=3.1 velocity=7.0
- joint r_upper_arm_z: limit lower=-2.6 upper=2.6 effort=0 velocity=0 -> lower=-2.6 upper=2.6 effort=3.1 velocity=7.0
- joint spine_z: limit lower=-2.6 upper=2.6 effort=0 velocity=0 -> lower=-2.6 upper=2.6 effort=3.1 velocity=7.0

Commit message: modified URDF

File: Hardware/URDF/robots/Heol_humanoid.URDF (robot description, URDF)
Before this commit: robot Heol_humanoid, 24 links, 23 joints
Links:
- link chest: mass 0.08200767006894 -> 0.0820076699949507
- link head: mass 0.0234153108401363 -> 0.023415330566188
- link l_shoulder: mass 0.00334368326561231 -> 0.0033436832656123
- link l_shoulder_motor: mass 0.03371809385647 -> 0.0337180938758863
- link l_upper_arm: mass 0.00334368326578747 -> 0.00334368326578746
- link r_ankle: mass 0.0401544687611881 -> 0.040154468761188
- link r_shoulder_motor: mass 0.0337180938758863 -> 0.03371809385647
Joints:
- removed joint r_hipy
- added joint r_hip_y: type revolute, parent pelvis, child r_hip, origin xyz=0.041652 -0.0188 0.0037433 rpy=1.5708 0 0, axis 0 -1 0, limit lower=-2.6 upper=2.6 effort=0 velocity=0

Commit message: update json

File: Hardware/URDF/robots/Heol_humanoid.URDF (robot description, URDF)
Before this commit: robot Heol_humanoid, 24 links, 23 joints
Joints:
- removed joint r_hipy
- added joint r_hip_y: type revolute, parent pelvis, child r_hip, origin xyz=0.041652 -0.0188 0.0037433 rpy=1.5708 0 0, axis 0 -1 0, limit lower=-2.6 upper=2.6 effort=3.1 velocity=7.0

Commit message: missed file

File: Hardware/URDF/robots/Heol_humanoid.URDF (robot description, URDF)
Before this commit: robot Heol_humanoid, 24 links, 23 joints
Links:
- link head: mass 0.023415330566188 -> 0.0234153106720677
- link l_ankle: mass 0.0401544687611881 -> 0.040154468761188
- link r_ankle: mass 0.040154468761188 -> 0.0401544687611881
- link r_knee: mass 0.00513087567995406 -> 0.00513087567995405
- link r_shoulder: mass 0.00334368326561429 -> 0.00334368326561428
Joints:
- removed joint r_hip_y
- added joint r_hipy: type revolute, parent pelvis, child r_hip, origin xyz=0.041652 -0.0188 0.0037433 rpy=1.5708 0 0, axis 0 -1 0, limit lower=-2.6 upper=2.6 effort=0 velocity=0
- joint chest_x: origin xyz=0 0.015 0 rpy=-1.5708 0 0 -> xyz=0 0.015 0 rpy=-1.5449 -8.1098E-17 -2.0871E-18
- joint head_z: origin xyz=0.00020517 -0.0021163 0.076016 rpy=1.5967 6.4765E-05 -6.3111E-05 -> xyz=0.0002 -0.00015034 0.076045 rpy=1.5708 4.9504E-11 -0.0025045
- joint l_ankle_x: origin xyz=0 0.045 0 rpy=3.4694E-16 0 3.1416 -> xyz=-0.056743 -0.0302 0.0096519 rpy=3.4694E-16 0 3.1416
- joint l_foot_y: origin xyz=0 0 -0.0002 rpy=2.949E-15 0 3.1416 -> xyz=-0.011743 -0.0752 -0.0098519 rpy=2.949E-15 0 3.1416
- joint l_forearm_y: origin xyz=0.018 0 0 rpy=3.1416 1.1102E-14 -1.5708 -> xyz=0.018 0 0 rpy=3.1416 0 -1.5708
- joint l_shoulder_motor_y: origin xyz=0.018 0 0 rpy=0 -7.8886E-31 0 -> xyz=0.018089 0 0 rpy=0 0 0
- joint l_shoulder_x: origin xyz=-0.0436 -0.00015034 0.051 rpy=1.5708 -1.3E-29 3.1416 -> xyz=-0.043511 -0.00015034 0.061 rpy=1.5967 1.7916E-17 3.1416
- joint l_upper_arm_z: origin xyz=0 -0.054 0 rpy=3.1416 2.0817E-15 -1.5708 -> xyz=0 -0.054 0 rpy=-3.1392 0 -1.5708
- joint r_ankle_x: origin xyz=0 -0.045 0 rpy=-3.1416 1.3878E-15 3.1416 -> xyz=0 -0.044 0 rpy=-3.1416 1.3878E-15 3.1416
- joint r_foot_y: origin xyz=0 0 -0.0002 rpy=1.3878E-15 8.3267E-15 3.1416 -> xyz=0 0 0 rpy=1.3878E-15 8.3267E-15 3.1416
- joint r_forearm_y: origin xyz=0.018 0 0 rpy=-3.1416 2.0817E-14 -1.5708 -> xyz=0.018 0 0 rpy=3.1416 0 -1.5708
- joint r_knee_x: origin xyz=0 -0.045 0 rpy=1.3878E-15 1.3878E-15 1.3482E-29 -> xyz=0 -0.046 0 rpy=1.3878E-15 1.3878E-15 1.3482E-29
- joint r_shoulder_motor_y: origin xyz=0.018089 0 0 rpy=-9.8608E-32 4.3368E-19 3.1416 -> xyz=0.018089 0 0 rpy=0 0 3.1416
- joint r_shoulder_x: origin xyz=0.043911 0.00010717 0.051 rpy=-1.5708 -1.6935E-18 0.0024405 -> xyz=0.043911 -0.00015034 0.061 rpy=-1.5967 5.5447E-11 2.1434E-09
- joint r_upper_arm_z: origin xyz=0 -0.054 0 rpy=-3.1392 6.9389E-16 -1.5708 -> xyz=0 -0.054 0 rpy=-3.1392 0 -1.5708
- joint spine_z: origin xyz=0.041652 -0.0728 0.058743 rpy=3.1416 0 0 -> xyz=0.041652 -0.0728 0.058743 rpy=3.1416 -0.0024405 1.4944E-19
