Commit message: modified URDF

File: Hardware/URDF/robots/Heol_humanoid.URDF (robot description, URDF)
Before this commit: robot Heol_humanoid, 24 links, 23 joints
Links:
- link chest: mass 0.0820076699949507 -> 0.082007665212002; geometry collision mesh filename=package://Heol_humanoid/meshes/chest.STL; visual mesh filename=package://Heol_humanoid/meshes/chest.STL
- link head: mass 0.0234153106720677 -> 0.0234154282160459; geometry collision mesh filename=package://Heol_humanoid/meshes/head.STL; visual mesh filename=package://Heol_humanoid/meshes/head.STL
- link l_ankle: geometry collision mesh filename=package://Heol_humanoid/meshes/l_ankle.STL; visual mesh filename=package://Heol_humanoid/meshes/l_ankle.STL
- link l_foot: geometry collision mesh filename=package://Heol_humanoid/meshes/l_foot.STL; visual mesh filename=package://Heol_humanoid/meshes/l_foot.STL
- link l_forearm: geometry collision mesh filename=package://Heol_humanoid/meshes/l_forearm.STL; visual mesh filename=package://Heol_humanoid/meshes/l_forearm.STL
- link l_hip: geometry collision mesh filename=package://Heol_humanoid/meshes/l_hip.STL; visual mesh filename=package://Heol_humanoid/meshes/l_hip.STL
- link l_hip_motor: geometry collision mesh filename=package://Heol_humanoid/meshes/l_hip_motor.STL; visual mesh filename=package://Heol_humanoid/meshes/l_hip_motor.STL
- link l_knee: mass 0.00513087567995406 -> 0.00513087567995407; geometry collision mesh filename=package://Heol_humanoid/meshes/l_knee.STL; visual mesh filename=package://Heol_humanoid/meshes/l_knee.STL
- link l_shoulder: mass 0.0033436832656123 -> 0.00334368326561229; geometry collision mesh filename=package://Heol_humanoid/meshes/l_shoulder.STL; visual mesh filename=package://Heol_humanoid/meshes/l_shoulder.STL
- link l_shoulder_motor: mass 0.0337180938758863 -> 0.03371809385647; geometry collision mesh filename=package://Heol_humanoid/meshes/l_shoulder_motor.STL; visual mesh filename=package://Heol_humanoid/meshes/l_shoulder_motor.STL
- link l_thigh: geometry collision mesh filename=package://Heol_humanoid/meshes/l_thigh.STL; visual mesh filename=package://Heol_humanoid/meshes/l_thigh.STL
- link l_upper_arm: mass 0.00334368326578746 -> 0.00334368326578747; geometry collision mesh filename=package://Heol_humanoid/meshes/l_upper_arm.STL; visual mesh filename=package://Heol_humanoid/meshes/l_upper_arm.STL
- link pelvis: geometry collision mesh filename=package://Heol_humanoid/meshes/pelvis.STL; visual mesh filename=package://Heol_humanoid/meshes/pelvis.STL
- link r_ankle: mass 0.0401544687611881 -> 0.040154468761188; geometry collision mesh filename=package://Heol_humanoid/meshes/r_ankle.STL; visual mesh filename=package://Heol_humanoid/meshes/r_ankle.STL
- link r_foot: geometry collision mesh filename=package://Heol_humanoid/meshes/r_foot.STL; visual mesh filename=package://Heol_humanoid/meshes/r_foot.STL
- link r_forearm: mass 0.0257657889801188 -> 0.0257657889801187; geometry collision mesh filename=package://Heol_humanoid/meshes/r_forearm.STL; visual mesh filename=package://Heol_humanoid/meshes/r_forearm.STL
- link r_hip: geometry collision mesh filename=package://Heol_humanoid/meshes/r_hip.STL; visual mesh filename=package://Heol_humanoid/meshes/r_hip.STL
- link r_hip_motor: geometry collision mesh filename=package://Heol_humanoid/meshes/r_hip_motor.STL; visual mesh filename=package://Heol_humanoid/meshes/r_hip_motor.STL
- link r_knee: mass 0.00513087567995405 -> 0.00513087567995406; geometry collision mesh filename=package://Heol_humanoid/meshes/r_knee.STL; visual mesh filename=package://Heol_humanoid/meshes/r_knee.STL
- link r_shoulder: mass 0.00334368326561428 -> 0.00334368326561429; geometry collision mesh filename=package://Heol_humanoid/meshes/r_shoulder.STL; visual mesh filename=package://Heol_humanoid/meshes/r_shoulder.STL
- link r_shoulder_motor: geometry collision mesh filename=package://Heol_humanoid/meshes/r_shoulder_motor.STL; visual mesh filename=package://Heol_humanoid/meshes/r_shoulder_motor.STL
- link r_thigh: geometry collision mesh filename=package://Heol_humanoid/meshes/r_thigh.STL; visual mesh filename=package://Heol_humanoid/meshes/r_thigh.STL
- link r_upper_arm: geometry collision mesh filename=package://Heol_humanoid/meshes/r_upper_arm.STL; visual mesh filename=package://Heol_humanoid/meshes/r_upper_arm.STL
- link spine: mass 0.0236192598262425 -> 0.0236192598262426; geometry collision mesh filename=package://Heol_humanoid/meshes/spine.STL; visual mesh filename=package://Heol_humanoid/meshes/spine.STL
Joints:
- joint chest_x: limit lower=-2.61799387799 upper=2.61799387799 effort=0.39 velocity=11.9 -> lower=-2.6 upper=2.6 effort=0 velocity=0; origin xyz=0 0.015 0 rpy=-1.5449 -8.1098E-17 -2.0871E-18 -> xyz=0 0.015 0 rpy=-1.5733 -2.2161E-16 5.4549E-19
- joint head_z: limit lower=-2.61799387799 upper=2.61799387799 effort=0.39 velocity=11.9 -> lower=-2.6 upper=2.6 effort=0 velocity=0; origin xyz=0.0002 -0.00015034 0.076045 rpy=1.5708 4.9504E-11 -0.0025045 -> xyz=0.0002 -0.00015034 0.075799 rpy=1.5708 6.1724E-06 -0.0025045
- joint l_ankle_x: limit lower=-2.61799387799 upper=2.61799387799 effort=0.39 velocity=11.9 -> lower=-2.6 upper=2.6 effort=0 velocity=0; origin xyz=-0.056743 -0.0302 0.0096519 rpy=3.4694E-16 0 3.1416 -> xyz=0 0.044 0 rpy=3.4694E-16 0 3.1416
- joint l_foot_y: limit lower=-2.61799387799 upper=2.61799387799 effort=0.39 velocity=11.9 -> lower=-2.6 upper=2.6 effort=0 velocity=0; origin xyz=-0.011743 -0.0752 -0.0098519 rpy=2.949E-15 0 3.1416 -> xyz=0 0 0 rpy=2.949E-15 0 3.1416
- joint l_forearm_y: limit lower=-2.61799387799 upper=2.61799387799 effort=0.39 velocity=11.9 -> lower=-2.6 upper=2.6 effort=0 velocity=0; origin xyz=0.018 0 0 rpy=3.1416 0 -1.5708 -> xyz=0.018 0 0 rpy=3.1416 6.9389E-16 -1.5708
- joint l_hip_motor_z: limit lower=-2.61799387799 upper=2.61799387799 effort=0.39 velocity=11.9 -> lower=-2.6 upper=2.6 effort=0 velocity=0
- joint l_hip_y: limit lower=-2.61799387799 upper=2.61799387799 effort=0.39 velocity=11.9 -> lower=-2.6 upper=2.6 effort=0 velocity=0
- joint l_knee_x: limit lower=-2.61799387799 upper=2.61799387799 effort=0.39 velocity=11.9 -> lower=-2.6 upper=2.6 effort=0 velocity=0; origin xyz=0 -0.045 0 rpy=-3.1416 0 0 -> xyz=0 -0.046 0 rpy=-3.1416 0 0
- joint l_shoulder_motor_y: limit lower=-2.61799387799 upper=2.61799387799 effort=0.39 velocity=11.9 -> lower=-2.6 upper=2.6 effort=0 velocity=0; origin xyz=0.018089 0 0 rpy=0 0 0 -> xyz=0.018089 0 0 rpy=9.8608E-32 -4.3368E-19 0
- joint l_shoulder_x: limit lower=-2.61799387799 upper=2.61799387799 effort=0.39 velocity=11.9 -> lower=-2.6 upper=2.6 effort=0 velocity=0; origin xyz=-0.043511 -0.00015034 0.061 rpy=1.5967 1.7916E-17 3.1416 -> xyz=-0.043511 -0.00015034 0.061 rpy=1.5683 -1.6926E-18 -3.1416
- joint l_thigh_x: limit lower=-2.61799387799 upper=2.61799387799 effort=0.39 velocity=11.9 -> lower=-2.6 upper=2.6 effort=0 velocity=0
- joint l_upper_arm_z: limit lower=-2.61799387799 upper=2.61799387799 effort=0.39 velocity=11.9 -> lower=-2.6 upper=2.6 effort=0 velocity=0; origin xyz=0 -0.054 0 rpy=-3.1392 0 -1.5708 -> xyz=0 -0.054 0 rpy=-3.1392 -6.9389E-16 -1.5708
- joint r_ankle_x: limit lower=-2.61799387799 upper=2.61799387799 effort=0.39 velocity=11.9 -> lower=-2.6 upper=2.6 effort=0 velocity=0
- joint r_foot_y: limit lower=-2.61799387799 upper=2.61799387799 effort=0.39 velocity=11.9 -> lower=-2.6 upper=2.6 effort=0 velocity=0
- joint r_forearm_y: limit lower=-2.61799387799 upper=2.61799387799 effort=0.39 velocity=11.9 -> lower=-2.6 upper=2.6 effort=0 velocity=0
- joint r_hip_motor_z: limit lower=-2.61799387799 upper=2.61799387799 effort=0.39 velocity=11.9 -> lower=-2.6 upper=2.6 effort=0 velocity=0
- joint r_hip_y: limit lower=-2.61799387799 upper=2.61799387799 effort=0.39 velocity=11.9 -> lower=-2.6 upper=2.6 effort=0 velocity=0
- joint r_knee_x: limit lower=-2.61799387799 upper=2.61799387799 effort=0.39 velocity=11.9 -> lower=-2.6 upper=2.6 effort=0 velocity=0
- joint r_shoulder_motor_y: limit lower=-2.61799387799 upper=2.61799387799 effort=0.39 velocity=11.9 -> lower=-2.6 upper=2.6 effort=0 velocity=0
- joint r_shoulder_x: limit lower=-2.61799387799 upper=2.61799387799 effort=0.39 velocity=11.9 -> lower=-2.6 upper=2.6 effort=0 velocity=0; origin xyz=0.043911 -0.00015034 0.061 rpy=-1.5967 5.5447E-11 2.1434E-09 -> xyz=0.043911 -0.00015034 0.061 rpy=-1.5683 -4.2352E-21 2.2291E-16
- joint r_thigh_x: limit lower=-2.61799387799 upper=2.61799387799 effort=0.39 velocity=11.9 -> lower=-2.6 upper=2.6 effort=0 velocity=0
- joint r_upper_arm_z: limit lower=-2.61799387799 upper=2.61799387799 effort=0.39 velocity=11.9 -> lower=-2.6 upper=2.6 effort=0 velocity=0
- joint spine_z: limit lower=-2.61799387799 upper=2.61799387799 effort=0.39 velocity=11.9 -> lower=-2.6 upper=2.6 effort=0 velocity=0
